Commit message: Modified and improved Multi-Vehicle node hierarchy for simulation

File: racecar1.xacro (robot description, xacro)
@@ -14,6 +14,6 @@
     <color rgba="0.2 0.2 0.2 1."/>
   </material>
-  <material name="purple">
-    <color rgba="1 0.57 1. 1."/>
+  <material name="blue">
+    <color rgba="0.3 0.57 1. 1."/>
   </material>
   <!-- Define a prefix property -->
@@ -25,5 +25,5 @@
         <box size="${wheelbase} ${width} ${height}"/>
       </geometry>
-      <material name="purple"/>
+      <material name="blue"/>
     </visual>
   </link>

File: racecar2.xacro (robot description, xacro)
@@ -1,5 +1,5 @@
 <?xml version="1.0"?>
 <!-- A simple model of the racecar for rviz -->
-<robot xmlns:xacro="http://www.ros.org/wiki/xacro" name="racecar1">
+<robot xmlns:xacro="http://www.ros.org/wiki/xacro" name="racecar2">
   <xacro:property name="wheelbase" value="0.5002" />
   <xacro:property name="width" value="0.3632" />
@@ -18,5 +18,5 @@
   </material>
   <!-- Define a prefix property -->
-  <xacro:property name="prefix" value="racecar1/" />
+  <xacro:property name="prefix" value="racecar2/" />
   <link name="${prefix}base_link">
     <visual>
